File: Atari 130XE.kicad_pcb (KiCad board)
At the start: 2 copper layers, 324.7 x 189 mm, 296 parts, among them J1 Power, J15 SIO_Port, J2 DIN-5_180degree, J3 Cartridge, J4 Joystick_Port, J5 Joystick_Port, J51 OS Type, J52 Conn_02x08_Odd_Even, J6 Keyboard, J7 SIMM_ON_OFF, Q1 2N3904, Q10 BC549, Q2 2N3904, Q3 2N3904, Q4 2N3906, Q6 2N3904, Q8 PN2222A, Q9 PN2222A, SW1 Switch_power_on, U1 PIA, U11 74LS74, U110 74AHC1G08, U111 74AHC1G08, U112 74AHC1G08, U113 74AHC1G08, U12 4050, U120 SIMM_exp_GAL, U121 DRAM_1MB_4bit, U122 DRAM_1MB_4bit, U123 74LS175, U124 74LS157, U13 74LS138, U14 MMU, U17 DRAM_4464, U18 DRAM_4464, U2 Antic, U21 NE555, U3 GTIA, U5 POKEY, U59 74HC74, U6 Sally, U60 74HC02, U61 74HC02, U62 4051, U63 4051, U7 27C512, U8 27C010, U9 Freddie, Y1 14,18757MHz, Y2 4.43MHz

Commit message: Crystal track
Parts:
- moved J51 83.3 mm to (261.6, 165.1), turned to 90 degrees
- moved C206 17.9 mm to (159.6, 173.3), turned to 270 degrees
- moved Q6 15.4 mm to (157.7, 163.6)
- moved FB3 14.3 mm to (156.0, 168.2)
- moved C111 12.0 mm to (177.9, 178.2), turned to 90 degrees
- moved C60 12.0 mm to (162.8, 173.3), turned to 270 degrees
- moved R37 10.2 mm to (179.4, 90.9), turned to 270 degrees
- moved R71 7.90 mm to (174.9, 178.2)
- moved L1 7.69 mm to (172.0, 168.1)
- moved C61 7.68 mm to (181.1, 173.2), turned to 270 degrees
- moved R73 7.42 mm to (169.1, 178.2)
- moved C59 7.21 mm to (166.1, 178.3)
- moved R72 6.63 mm to (146.8, 178.4)
- moved R70 6.48 mm to (149.6, 178.4)
- moved C28 5.52 mm to (158.6, 155.8), turned to 180 degrees
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Routing:
- net GND: track 534.3 -> 734.2 mm
- net R\W: track 227.4 -> 403.3 mm, vias 5 -> 7
- net RST: track 365.1 -> 526.2 mm, vias 7 -> 8
- net Net-(C48-Pad2): track 0.00 -> 141.9 mm, vias 0 -> 4
- net Net-(Q6-Pad3): track 0.00 -> 126.4 mm, vias 0 -> 1
- net RD5: track 183.6 -> 297.8 mm, vias 2 -> 4
- net Net-(C206-Pad1): track 0.00 -> 112.4 mm, vias 0 -> 2
- net SOUND: track 194.3 -> 290.6 mm
- net OSC: track 0.00 -> 92.2 mm
- net Net-(L66-Pad1): track 0.00 -> 76.9 mm
- net Net-(Q10-Pad2): track 0.00 -> 62.2 mm, vias 0 -> 1
- net Net-(Q3-Pad2): track 0.00 -> 60.5 mm
- net Net-(U112-Pad1): track 58.8 -> 0.00 mm, vias 2 -> 0
- net Net-(C47-Pad2): track 0.00 -> 43.9 mm
- net BELL: track 139.5 -> 177.8 mm
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- added copper zone on F.Cu, net GND

Commit message: Track
Parts:
- moved R12 21.4 mm to (271.7, 100.8), turned to 180 degrees
- moved C26 3.35 mm to (270.7, 103.2), turned to 270 degrees
- moved U13 2.31 mm to (274.0, 111.2)
- moved C1 0.28 mm to (190.8, 90.9)
Connections:
- C42 pad 2: Net-(C40-Pad1) -> GND
Routing:
- net BO2: track 133.6 -> 352.2 mm, vias 3 -> 8
- net R\W: track 403.3 -> 517.6 mm, vias 7 -> 6
- net RST: track 526.2 -> 469.7 mm
- net A10: track 346.2 -> 379.3 mm, vias 4 -> 6
- net A2: track 495.1 -> 463.0 mm
- net +5VA: track 55.3 -> 79.7 mm
- net Net-(C40-Pad1): track 46.2 -> 23.7 mm
- net SOUND: track 290.6 -> 283.2 mm
- net A3: track 460.2 -> 453.5 mm, vias 10 -> 7
- net BELL: track 177.8 -> 171.5 mm
- net O1: track 30.6 -> 25.3 mm, vias 1 -> 2
- net Net-(R134-Pad2): track 181.9 -> 176.7 mm, vias 3 -> 1
- net VCC: track 1043.4 -> 1047.8 mm, vias 17 -> 15
- net A5: track 328.7 -> 324.8 mm
- net A12_cart: track 40.3 -> 43.8 mm
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