File: Atari 130XE.kicad_pcb (KiCad board)
At the start: 2 copper layers, 324.7 x 189 mm, 296 parts, among them J1 Power, J15 SIO_Port, J2 DIN-5_180degree, J3 Cartridge, J4 Joystick_Port, J5 Joystick_Port, J51 OS Type, J52 Conn_02x08_Odd_Even, J6 Keyboard, J7 SIMM_ON_OFF, Q1 2N3904, Q10 BC549, Q2 2N3904, Q3 2N3904, Q4 2N3906, Q6 2N3904, Q8 PN2222A, Q9 PN2222A, SW1 Switch_power_on, U1 PIA, U11 74LS74, U110 74AHC1G08, U111 74AHC1G08, U112 74AHC1G08, U113 74AHC1G08, U12 4050, U120 SIMM_exp_GAL, U121 DRAM_1MB_4bit, U122 DRAM_1MB_4bit, U123 74LS175, U124 74LS157, U13 74LS138, U14 MMU, U17 DRAM_4464, U18 DRAM_4464, U2 Antic, U21 NE555, U3 GTIA, U5 POKEY, U59 74HC74, U6 Sally, U60 74HC02, U61 74HC02, U62 4051, U63 4051, U7 27C512, U8 27C010, U9 Freddie, Y1 14,18757MHz, Y2 4.43MHz

Commit message: Track
Parts:
- R4, R6, R7: moved to F.Cu
- moved R2 104.6 mm to (286.3, 99.0)
- moved R3 104.6 mm to (286.3, 96.7)
- moved U110 104.6 mm to (281.7, 98.0)
- moved C106 104.6 mm to (290.7, 94.7)
- moved C112 104.6 mm to (281.6, 94.7)
- moved U112 104.6 mm to (290.8, 98.0)
- moved C1 67.9 mm to (258.7, 89.0)
- moved C103 64.4 mm to (99.7, 94.5), turned to 90 degrees
- moved R148 56.0 mm to (102.5, 99.7), turned to 90 degrees
- moved R4 30.6 mm to (179.6, 85.2), turned to 270 degrees
- moved R7 28.0 mm to (177.2, 85.2), turned to 270 degrees
- moved R6 25.4 mm to (174.9, 85.2), turned to 270 degrees
- moved U13 5.43 mm to (279.0, 113.4)
- moved C100 0.08 mm to (122.0, 89.5)
- moved C101 0.08 mm to (113.7, 94.5)
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Routing:
- net RD4: track 14.0 -> 241.8 mm, vias 0 -> 4
- net S4: track 0.00 -> 198.8 mm, vias 0 -> 3
- net Net-(U13-Pad4): track 0.00 -> 186.2 mm, vias 0 -> 1
- net S5: track 0.00 -> 172.8 mm, vias 0 -> 4
- net A15: track 81.4 -> 227.8 mm, vias 1 -> 3
- net A14: track 79.8 -> 221.1 mm, vias 2 -> 4
- net HALT: track 111.9 -> 250.3 mm, vias 4 -> 8
- net REF: track 46.2 -> 176.3 mm, vias 0 -> 2
- net O2: track 137.1 -> 260.0 mm, vias 2 -> 4
- net BELL: track 171.5 -> 235.2 mm
- net VCC: track 1047.8 -> 1000.0 mm, vias 15 -> 13
- net A10: track 379.3 -> 418.6 mm, vias 6 -> 7
- net BO2: track 352.2 -> 389.6 mm, vias 8 -> 12
- net Net-(Q10-Pad2): track 62.2 -> 28.3 mm, vias 1 -> 0
- net NMI: track 29.1 -> 55.7 mm, vias 0 -> 1
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
Commit message: track
Parts:
- removed C106, C112, C113: 100n, Capacitor_SMD:C_0603_1608Metric_Pad1.05x0.95mm_HandSolder
- removed C107: 100nF, Capacitor_SMD:C_0603_1608Metric_Pad1.05x0.95mm_HandSolder
- removed U110, U111, U112, U113: 74AHC1G08, Package_TO_SOT_SMD:SOT-23-5_HandSoldering
- added U10: 74LS08, Package_DIP:DIP-14_W7.62mm_Socket_LongPads, F.Cu at (278.9, 100.3)
- U13: footprint Package_DIP:DIP-16_W7.62mm_Socket -> Package_DIP:DIP-16_W7.62mm_Socket_LongPads
- moved C25 225.6 mm to (275.6, 92.2), turned to 270 degrees
- moved FB4 21.8 mm to (288.5, 77.6), turned to 180 degrees
- moved R3 16.1 mm to (270.5, 93.6), turned to 90 degrees
- moved C97 14.6 mm to (286.8, 90.0), turned to 90 degrees
- moved R2 14.6 mm to (272.8, 93.6), turned to 90 degrees
- moved R132 12.8 mm to (284.0, 88.5), turned to 90 degrees
- moved R133 12.3 mm to (281.5, 88.5), turned to 90 degrees
- moved C1 10.5 mm to (265.2, 80.7)
- moved FB5 8.89 mm to (288.5, 81.5)
- moved C96 7.78 mm to (278.7, 89.9), turned to 90 degrees
- moved FB10 6.04 mm to (314.7, 87.5)
- moved FB11 6.04 mm to (314.7, 92.2)
- moved R12 6.00 mm to (272.7, 106.7), turned to 90 degrees
- moved C26 5.31 mm to (275.6, 105.3)
Routing:
- net Net-(R132-Pad1): track 0.00 -> 232.5 mm, vias 0 -> 4
- net Net-(R133-Pad1): track 0.00 -> 229.1 mm, vias 0 -> 4
- net OS: track 7.94 -> 133.3 mm, vias 0 -> 3
- net LP: track 0.00 -> 117.8 mm, vias 0 -> 1
- net GTIA: track 0.00 -> 108.3 mm, vias 0 -> 2
- net Net-(U10-Pad4): track 0.00 -> 103.1 mm, vias 0 -> 1
- net O2: track 260.0 -> 331.8 mm
- net PIA: track 0.00 -> 70.5 mm, vias 0 -> 2
- net O0: track 0.00 -> 55.8 mm
- net A8: track 295.7 -> 345.5 mm, vias 4 -> 5
- net A9: track 307.5 -> 355.6 mm, vias 6 -> 7
- net GND: track 730.4 -> 765.0 mm
- net Net-(U10-Pad10): track 0.00 -> 23.5 mm, vias 0 -> 1
- net R\W: track 518.5 -> 541.8 mm, vias 5 -> 6
- net Net-(R12-Pad1): track 0.00 -> 22.1 mm
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
Commit message: Track
Parts:
- R139: moved to B.Cu
- moved R83 7.86 mm to (306.6, 96.1), turned to 180 degrees
- moved R88 7.73 mm to (306.6, 98.7), turned to 180 degrees
- moved J51 5.68 mm to (266.7, 162.6), turned to 270 degrees
- moved R139 5.22 mm to (271.1, 195.2)
- moved Q1 0.34 mm to (176.2, 104.3)
Routing:
- net GND: track 765.0 -> 1073.7 mm, vias 119 -> 108
- net SIOAUDIO: track 0.00 -> 250.3 mm, vias 0 -> 4
- net A6: track 205.9 -> 364.2 mm, vias 1 -> 8
- net BASC_cart: track 14.8 -> 161.1 mm, vias 2 -> 8
- net A13_cart: track 0.00 -> 127.6 mm, vias 0 -> 6
- net TRIG1: track 0.00 -> 123.8 mm
- net VCC: track 1005.1 -> 1118.1 mm, vias 13 -> 14
- net Net-(R132-Pad1): track 232.5 -> 123.5 mm, vias 4 -> 3
- net Net-(J51-Pad3): track 0.00 -> 103.5 mm, vias 0 -> 2
- net TRIG0: track 0.00 -> 96.4 mm, vias 0 -> 1
- net Net-(J51-Pad4): track 0.00 -> 92.2 mm, vias 0 -> 2
- net Net-(C48-Pad2): track 145.3 -> 207.5 mm
- net CCTL: track 208.5 -> 267.8 mm, vias 2 -> 4
- net READY: track 51.5 -> 105.3 mm
- net O0: track 55.8 -> 106.0 mm, vias 0 -> 1
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
Commit message: Track
Parts:
- moved C24 169.2 mm to (228.0, 125.4)
- moved C1 55.4 mm to (213.1, 99.6), turned to 180 degrees
Connections:
- U3 pad 27: +5VA -> VCC
Routing:
- net VCC: track 1118.1 -> 1220.1 mm, vias 14 -> 20
- net R\W: track 541.8 -> 642.9 mm, vias 6 -> 7
- net GND: track 1073.7 -> 1122.3 mm
- net BELL: track 235.8 -> 277.0 mm, vias 2 -> 4
- net SOUND: track 281.8 -> 317.7 mm, vias 2 -> 4
- net HALT: track 252.7 -> 285.3 mm
- net +5VA: track 79.7 -> 55.3 mm
- net BASC_cart: track 161.1 -> 143.1 mm, vias 8 -> 6
- net GTIA: track 108.6 -> 125.7 mm, vias 2 -> 4
- net A6: track 364.2 -> 350.9 mm, vias 8 -> 6
- net A13_cart: track 127.6 -> 114.3 mm, vias 6 -> 4
- net A1: track 515.4 -> 524.4 mm, vias 7 -> 8
- net OS: track 133.3 -> 140.9 mm, vias 3 -> 4
- net Net-(R132-Pad1): track 123.5 -> 129.7 mm
- net Net-(R133-Pad1): track 228.3 -> 222.1 mm
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
Commit message: Track
Parts:
- R29, R4, R6, R7: footprint Resistor_SMD:R_1206_3216Metric_Pad1.42x1.75mm_HandSolder -> Atari:R_Axial_DIN0207_L3.6mm_D2.2mm_P10.16mm_Horizontal
- moved R29 25.8 mm to (96.8, 89.5), turned to 270 degrees
- moved R4 14.1 mm to (165.8, 88.2), turned to 90 degrees
- moved R7 9.20 mm to (168.5, 88.2), turned to 90 degrees
- moved R6 4.71 mm to (171.3, 88.2), turned to 90 degrees
Routing:
- net GND: track 1122.3 -> 2004.3 mm, vias 108 -> 183
- net VCC: track 1220.1 -> 1644.7 mm, vias 20 -> 35
- net CHROMA: track 0.00 -> 129.9 mm, vias 0 -> 1
- net +5VA: track 55.3 -> 148.4 mm
- net AUDIO: track 0.00 -> 74.4 mm
- net PB5: track 333.0 -> 271.4 mm
- net PB6: track 348.6 -> 289.0 mm
- net PB7: track 353.3 -> 294.3 mm
- net PB1: track 337.0 -> 279.8 mm
- net COMPOSITE: track 2.39 -> 53.5 mm
- net Net-(R29-Pad1): track 17.2 -> 48.7 mm
- net BASIC: track 215.7 -> 186.4 mm, vias 4 -> 2
- net NMI: track 52.9 -> 81.2 mm
- net MONO: track 0.00 -> 27.6 mm
- net IRQ: track 245.9 -> 270.4 mm
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- added copper zone on B.Cu, net GND

Commit message: Track
Parts:
- Q1, Q2, Q3, Q6, Q8, Q9: footprint Package_TO_SOT_THT:TO-92 -> Package_TO_SOT_THT:TO-92_Inline
- moved R36 10.2 mm to (182.1, 101.1), turned to 90 degrees
- moved D2 10.2 mm to (176.8, 91.0), turned to 270 degrees
- moved Q1 3.11 mm to (173.2, 105.3), turned to 0 degrees
Routing:
- net GND: track 2004.3 -> 2025.9 mm
- net +5VA: track 148.4 -> 159.5 mm
- net Net-(C45-Pad2): track 15.3 -> 24.8 mm
- net Net-(C45-Pad1): track 14.7 -> 8.63 mm
- net Net-(C48-Pad2): track 211.9 -> 207.1 mm
- net OS: track 140.9 -> 137.1 mm
- net RD5: track 298.0 -> 296.6 mm
- net Net-(Q2-Pad2): track 9.05 -> 7.77 mm
- net Net-(Q3-Pad1): track 33.1 -> 31.9 mm
- net Net-(Q6-Pad2): track 37.3 -> 38.6 mm
- net Net-(L66-Pad2): track 5.09 -> 3.82 mm
- net Net-(C44-Pad1): track 9.93 -> 11.1 mm

Commit message: Track OS and Basic
Parts:
- removed J51: OS Type, Connector_PinHeader_2.54mm:PinHeader_2x03_P2.54mm_Vertical
- removed J52: Conn_02x08_Odd_Even, Connector_PinHeader_2.54mm:PinHeader_2x08_P2.54mm_Vertical
- added J10: Os Type, Connector_PinHeader_2.54mm:PinHeader_2x06_P2.54mm_Vertical, F.Cu at (257.9, 173.2)
- added J11: Os Type, Connector_PinHeader_2.54mm:PinHeader_1x06_P2.54mm_Vertical, F.Cu at (257.9, 168.1)
- added J8: Basic_Sel, Connector_PinHeader_2.54mm:PinHeader_1x04_P2.54mm_Vertical, F.Cu at (246.3, 168.1)
- added J9: Basic_Sel, Connector_PinHeader_2.54mm:PinHeader_2x04_P2.54mm_Vertical, F.Cu at (246.3, 173.2)
- U7: value 27C512 -> 27C040; footprint Package_DIP:DIP-28_W15.24mm_LongPads -> Package_DIP:DIP-32_W15.24mm_Socket_LongPads
- moved U7 0.23 mm to (195.0, 191.8)
Connections:
- U7 pad 1: Net-(J51-Pad3) -> OSA19
- U7 pad 10: A0 -> A2
- U7 pad 11: D0 -> A1
- U7 pad 12: D1 -> A0
- U7 pad 13: D2 -> D0
- U7 pad 14: GND -> D1
- U7 pad 15: D3 -> D2
- U7 pad 16: D4 -> GND
- U7 pad 17: D5 -> D3
- U7 pad 18: D6 -> D4
- U7 pad 19: D7 -> D5
- U7 pad 2: A12 -> OSA16
- U7 pad 20: OS -> D6
- U7 pad 21: A10 -> D7
- U7 pad 23: A11 -> A10
- U7 pad 24: A9 -> OS
- U7 pad 25: A8 -> A11
- U7 pad 26: A13 -> A9
- U7 pad 27: Net-(J51-Pad4) -> A8
- U7 pad 28: VCC -> A13
- U7 pad 3: A7 -> OSA15
- U7 pad 4: A6 -> A12
- U7 pad 5: A5 -> A7
- U7 pad 6: A4 -> A6
- U7 pad 7: A3 -> A5
- U7 pad 8: A2 -> A4
- U7 pad 9: A1 -> A3
Routing:
- net Net-(J51-Pad3): track 104.1 -> 0.00 mm, vias 2 -> 0
- net +5VA: track 159.5 -> 262.0 mm
- net Net-(J51-Pad4): track 91.7 -> 0.00 mm, vias 2 -> 0
- net OSA19: track 0.00 -> 90.3 mm, vias 0 -> 2
- net GND: track 2025.9 -> 2115.2 mm
- net OSA16: track 0.00 -> 82.4 mm, vias 0 -> 1
- net OSA18: track 0.00 -> 80.3 mm, vias 0 -> 1
- net OSA15: track 0.00 -> 76.5 mm, vias 0 -> 1
- net OSA17: track 0.00 -> 75.6 mm, vias 0 -> 1
- net OSA14: track 0.00 -> 62.5 mm
- net VCC: track 1644.7 -> 1681.1 mm, vias 35 -> 36
- net R\W: track 627.9 -> 606.1 mm, vias 9 -> 7
- net Net-(R45-Pad2): track 44.1 -> 51.2 mm
- net A10: track 421.6 -> 415.0 mm, vias 7 -> 6
- net A14_sel: track 83.3 -> 76.9 mm
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
Commit message: Finished GND
Parts:
- added C106: 1nF, Capacitor_THT:C_Disc_D5.0mm_W2.5mm_P5.00mm, F.Cu at (83.9, 68.8)
- added C107: 1nF, Capacitor_THT:C_Disc_D5.0mm_W2.5mm_P5.00mm, F.Cu at (99.2, 68.8)
- added C98: 100uF, Capacitor_THT:CP_Radial_D6.3mm_P2.50mm, F.Cu at (126.0, 123.0)
- added J12: Conn_01x03, Connector_PinHeader_2.54mm:PinHeader_1x03_P2.54mm_Vertical, F.Cu at (154.3, 63.1)
- added J13: Conn_01x03, Connector_PinHeader_2.54mm:PinHeader_1x03_P2.54mm_Vertical, F.Cu at (171.9, 63.1)
- added J14: Conn_01x06, Connector_PinHeader_2.54mm:PinHeader_1x06_P2.54mm_Vertical, F.Cu at (72.0, 193.0)
- added J16: Conn_01x05, Connector_PinHeader_2.54mm:PinHeader_1x05_P2.54mm_Vertical, F.Cu at (72.1, 216.7)
- added J17: Conn_01x04, Connector_PinHeader_2.54mm:PinHeader_1x04_P2.54mm_Vertical, F.Cu at (297.8, 100.1)
- added J18: Pin, Atari:Pin, F.Cu at (154.5, 127.2)
- added J19: Pin, Atari:Pin, F.Cu at (159.6, 178.3)
- added J20: Pin, Atari:Pin, F.Cu at (162.8, 178.3)
- added J21: Pin, Atari:Pin, F.Cu at (166.1, 178.3)
- added J22: Pin, Atari:Pin, F.Cu at (181.0, 178.3)
- added J23: Pin, Atari:Pin, F.Cu at (177.9, 178.3)
- added J24: Pin, Atari:Pin, F.Cu at (173.3, 106.7)
- added J25: Pin, Atari:Pin, F.Cu at (171.9, 91.0)
- added J26: Pin, Atari:Pin, F.Cu at (168.9, 91.0)
- added J27: Pin, Atari:Pin, F.Cu at (165.8, 91.0)
- added J28: Pin, Atari:Pin, F.Cu at (162.8, 91.0)
- added J29: Pin, Atari:Pin, F.Cu at (135.9, 88.2)
- C39: footprint Capacitor_SMD:C_1206_3216Metric_Pad1.42x1.75mm_HandSolder -> Capacitor_THT:C_Disc_D5.0mm_W2.5mm_P5.00mm
- Q4: footprint Package_TO_SOT_THT:TO-92 -> Package_TO_SOT_THT:TO-92_Inline
- R16, R17: footprint Resistor_THT:R_Axial_DIN0207_L6.3mm_D2.5mm_P10.16mm_Horizontal -> Atari:R_Axial_DIN0207_L3.6mm_D2.2mm_P10.16mm_Horizontal
- R95, R96, R97, R98: footprint Resistor_SMD:R_1206_3216Metric_Pad1.42x1.75mm_HandSolder -> Atari:R_Axial_DIN0207_L3.6mm_D2.2mm_P10.16mm_Horizontal
- moved R98 15.7 mm to (127.7, 78.0), turned to 270 degrees
- moved R97 12.2 mm to (130.3, 78.0), turned to 270 degrees
- moved Q9 9.13 mm to (143.0, 87.8)
- moved Q1 8.05 mm to (165.2, 105.2)
- moved Q4 7.43 mm to (307.7, 102.1)
- moved R96 6.81 mm to (133.0, 88.2), turned to 90 degrees
- moved R95 6.37 mm to (138.8, 78.0), turned to 270 degrees
- moved C59 5.12 mm to (166.1, 173.2)
- moved C111 5.12 mm to (177.9, 173.1)
- moved C206 5.12 mm to (159.5, 168.2)
- moved C60 5.12 mm to (162.8, 168.2)
- moved C61 5.12 mm to (181.0, 168.1)
- moved R147 3.07 mm to (122.2, 89.5)
- moved C39 2.97 mm to (135.9, 83.0), turned to 90 degrees
- moved C100 2.59 mm to (119.4, 89.5)
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Routing:
- net VCC: track 1681.1 -> 1770.0 mm, vias 36 -> 41
- net GND: track 2115.2 -> 2174.8 mm, vias 183 -> 218
- net O2: track 368.9 -> 399.2 mm
- net AUDIO: track 73.1 -> 98.3 mm, vias 0 -> 1
- net BO2: track 394.0 -> 412.0 mm
- net Net-(R88-Pad1): track 114.4 -> 100.8 mm, vias 3 -> 2
- net CHROMA: track 129.9 -> 117.8 mm
- net COMPOSITE: track 53.5 -> 43.0 mm
- net O0: track 105.9 -> 114.8 mm
- net Net-(Q9-Pad1): track 3.43 -> 11.8 mm
- net MONO: track 27.6 -> 35.7 mm
- net Net-(C39-Pad2): track 6.29 -> 14.1 mm
- net Net-(C39-Pad1): track 8.32 -> 16.1 mm
- net Net-(C44-Pad1): track 11.1 -> 18.6 mm
- net Net-(C206-Pad1): track 110.6 -> 103.5 mm
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Other:
- board text added: "4,43MHz"
- board text added: "74LS138"
- board text added: "74LS157"
- board text added: "74LS175"
- board text added: "74LS74"
- board text added: "75LS08"
- board text added: "A12"
- board text added: "A14"
- board text added: "A15"
- board text added: "A16"
- board text added: "ANTIC"
- board text added: "AUDIO"
- board text added: "Atari 65XE with extra RAM by Jacek Binkul - 11.2020"
- board text added: "BASIC"
- board text added: "BASIC SELECT"
- board text added: "CAS"
- board text added: "CHROMA"
- board text added: "COMPOSITE"
- board text added: "Casinh"
- board text added: "DRAM 1MB 4bit"
- board text added: "DRAM 4464"
- board text added: "Extsel"
- board text added: "FREDDIE"
- board text added: "GAL SIMM Expansion"
- board text added: "GND"
- board text added: "GTIA"
- board text added: "Keyboard"
- board text added: "MMU"
- board text added: "MONO"
- board text added: "O2"
- board text added: "OS"
- board text added: "OS SELECT"
- board text added: "OSA14"
- board text added: "OSA15"
- board text added: "OSA16"
- board text added: "OSA17"
- board text added: "OSA18"
- board text added: "OSA19"
- board text added: "OSC"
- board text added: "PIA"
- board text added: "POKEY"
- board text added: "Q2"
- board text added: "R/W"
- board text added: "RAS"
- board text added: "SALLY"
- board text added: "VCC"
- board text added: "WRT"
- board text removed: "Atari 65XE with extra RAM by Jacek Binkul - 07.2020"
