File: Atari 130XE.kicad_pcb (KiCad board)
At the start: 2 copper layers, 324.7 x 189 mm, 311 parts, among them J1 Power, J10 Os Type, J11 Os Type, J12 Conn_01x03, J13 Conn_01x03, J14 Conn_01x06, J15 SIO_Port, J16 Conn_01x05, J17 Conn_01x04, J18 Pin, J19 Pin, J2 DIN-5_180degree, J20 Pin, J21 Pin, J22 Pin, J23 Pin, J24 Pin, J25 Pin, J26 Pin, J27 Pin, J28 Pin, J29 Pin, J3 Cartridge, J4 Joystick_Port, J5 Joystick_Port, J6 Keyboard, J7 SIMM_ON_OFF, J8 Basic_Sel, J9 Basic_Sel, Q1 2N3904, Q10 BC549, Q2 2N3904, Q3 2N3904, Q4 2N3906, Q6 2N3904, Q8 PN2222A, Q9 PN2222A, SW1 Switch_power_on, U1 PIA, U10 74LS08, U11 74LS74, U12 4050, U120 SIMM_exp_GAL, U121 DRAM_1MB_4bit, U122 DRAM_1MB_4bit, U123 74LS175, U124 74LS157, U13 74LS138, U14 MMU, U17 DRAM_4464, U18 DRAM_4464, U2 Antic, U21 NE555, U3 GTIA, U5 POKEY, U59 74HC74, U6 Sally, U60 74HC02, U61 74HC02, U62 4051, U63 4051, U7 27C040, U8 27C010, U9 Freddie, Y1 14,18757MHz, Y2 4.43MHz

Commit message: Gerber
Parts:
- C34: footprint Capacitor_SMD:CP_Elec_6.3x5.3 -> Capacitor_THT:CP_Radial_D5.0mm_P2.00mm
- R1: footprint Resistor_SMD:R_1206_3216Metric_Pad1.42x1.75mm_HandSolder -> Atari:R_Axial_DIN0207_L3.6mm_D2.2mm_P10.16mm_Horizontal
- moved R1 3.61 mm to (56.1, 197.0)
- moved C34 0.56 mm to (298.1, 81.2)
Connections:
- J9 pad 4: A16_sel -> A14_sel
- J9 pad 8: A14_sel -> A16_sel
Routing:
- net GND: track 2174.8 -> 1935.9 mm, vias 218 -> 246
- net A14_sel: track 76.9 -> 70.9 mm, vias 3 -> 4
- net A16_sel: track 61.6 -> 66.4 mm
- net RA5: track 127.1 -> 123.9 mm
- net Net-(R88-Pad1): track 100.8 -> 103.7 mm, vias 2 -> 3
- net A7: track 291.9 -> 289.2 mm
- net RA6: track 130.0 -> 127.6 mm
- net A6: track 349.8 -> 347.5 mm
- net A8: track 346.5 -> 344.3 mm
- net READY: track 105.3 -> 107.5 mm, vias 1 -> 0
- net RD4: track 241.8 -> 239.9 mm
- net A9: track 355.7 -> 353.9 mm
- net RA7: track 147.6 -> 145.8 mm
- net A5: track 328.0 -> 326.3 mm
- net D6: track 514.4 -> 513.3 mm
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Other:
- board text added: "1 MB"
- board text added: "512kB"
- board text added: "Atari 65XE with 1MB RAM by Jacek Binkul - 11.2020"
- board text added: "CD4050"
- board text added: "CD4051"
- board text added: "OFF"
- board text added: "ON"
- board text removed: "Atari 65XE with extra RAM by Jacek Binkul - 11.2020"

Commit message: Improve gerber
Routing:
- net GND: track 1935.9 -> 1918.3 mm
- net Net-(R135-Pad2): track 182.2 -> 180.7 mm
- net Net-(R134-Pad2): track 177.0 -> 175.5 mm
- net Net-(R136-Pad2): track 188.1 -> 186.6 mm
- net A7: track 289.2 -> 290.6 mm
- net A13: track 387.1 -> 388.3 mm
- net A5: track 326.3 -> 327.5 mm
- net A4: track 345.0 -> 346.2 mm
- net A6: track 347.5 -> 348.7 mm
- net D2: track 489.3 -> 488.2 mm
- net D6: track 513.3 -> 514.4 mm
- net A14: track 219.4 -> 220.5 mm
- net A15: track 224.9 -> 223.8 mm
- net Net-(L6-Pad1): track 84.9 -> 83.8 mm
- net A12: track 526.2 -> 527.2 mm
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