File: Reset i sound.sch (KiCad schematic (older format))
At the start: 7 parts, among them U21 NE555

Commit message: Track
Connections:
- net GND: now also C42.2
- net at C40.1, D6.1 (K), R93.1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: no longer C42.2
Changed lines of the file:
@@
-$EndComp
-$Comp
-L Device:C C42
-U 1 1 5E77A0C8
-P 4950 4250
-F 0 "C42" H 5065 4296 50  0000 L CNN
-F 1 "100n" H 5065 4205 50  0000 L CNN
-F 2 "Capacitor_SMD:C_1206_3216Metric_Pad1.42x1.75mm_HandSolder" H 4988 4100 50  0001 C CNN
-F 3 "~" H 4950 4250 50  0001 C CNN
-	1    4950 4250
-	1    0    0    -1
 $EndComp
 $Comp
@@
 $EndComp
 Wire Wire Line
-	3600 4500 3600 4700
+	3600 4500 3600 4575
 $Comp
 L power:VCC #PWR0230
@@
 Wire Wire Line
 	4950 3400 4950 4100
+$Comp
+L Device:C C42
+U 1 1 5E77A0C8
+P 4950 4250
+F 0 "C42" H 5065 4296 50  0000 L CNN
+F 1 "100n" H 5065 4205 50  0000 L CNN
+F 2 "Capacitor_SMD:C_1206_3216Metric_Pad1.42x1.75mm_HandSolder" H 4988 4100 50  0001 C CNN
+F 3 "~" H 4950 4250 50  0001 C CNN
+	1    4950 4250
+	1    0    0    -1
+$EndComp
 Wire Wire Line
-	4450 4950 4950 4950
+	3600 4575 4950 4575
 Wire Wire Line
-	4950 4950 4950 4400
-Connection ~ 4450 4950
+	4950 4575 4950 4400
+Connection ~ 3600 4575
+Wire Wire Line
+	3600 4575 3600 4700
 $EndSCHEMATC
