File: Sally and Antic.sch (KiCad schematic (older format))
At the start: 11 parts, among them U112 74AHC1G08, U2 Antic, U6 Sally

Commit message: track
Parts:
- removed C106: 100n, Capacitor_SMD:C_0603_1608Metric_Pad1.05x0.95mm_HandSolder, symbol Device:C
- removed U112: 74AHC1G08, Package_TO_SOT_SMD:SOT-23-5_HandSoldering, symbol 74xGxx:74AHC1G08
- added U10: 74LS08, Package_DIP:DIP-14_W7.62mm_Socket_LongPads, symbol 74xx:74LS08
Connections:
- net GND: now also U10.7 (GND)
- net O0: now also U10.6
- net VCC: now also U10.14 (VCC)
- net at U2.34 (O0): now also U10.4, U10.5
Changed lines of the file:
@@
 $EndComp
 $Comp
-L 74xGxx:74AHC1G08 U112
-U 1 1 5F80E771
-P 9175 3450
-F 0 "U112" H 9350 3625 50  0000 C CNN
-F 1 "74AHC1G08" H 8875 3625 50  0000 C CNN
-F 2 "Package_TO_SOT_SMD:SOT-23-5_HandSoldering" H 9175 3450 50  0001 C CNN
-F 3 "http://www.ti.com/lit/sg/scyt129e/scyt129e.pdf" H 9175 3450 50  0001 C CNN
-	1    9175 3450
+L 74xx:74LS08 U10
+U 2 1 5FA66C3F
+P 9125 3450
+F 0 "U10" H 9125 3775 50  0000 C CNN
+F 1 "74LS08" H 9125 3684 50  0000 C CNN
+F 2 "Package_DIP:DIP-14_W7.62mm_Socket_LongPads" H 9125 3450 50  0001 C CNN
+F 3 "http://www.ti.com/lit/gpn/sn74LS08" H 9125 3450 50  0001 C CNN
+	2    9125 3450
+	1    0    0    -1
+$EndComp
+Wire Wire Line
+	8800 3450 8800 3350
+Wire Wire Line
+	8800 3350 8825 3350
+Wire Wire Line
+	8800 3450 8800 3550
+Wire Wire Line
+	8800 3550 8825 3550
+Connection ~ 8800 3450
+$Comp
+L 74xx:74LS08 U10
+U 5 1 5FA6BF1F
+P 5125 6400
+F 0 "U10" H 5355 6446 50  0000 L CNN
+F 1 "74LS08" H 5355 6355 50  0000 L CNN
+F 2 "Package_DIP:DIP-14_W7.62mm_Socket_LongPads" H 5125 6400 50  0001 C CNN
+F 3 "http://www.ti.com/lit/gpn/sn74LS08" H 5125 6400 50  0001 C CNN
+	5    5125 6400
 	1    0    0    -1
 $EndComp
 $Comp
-L Device:C C106
-U 1 1 5F80F75F
-P 9800 3450
-F 0 "C106" H 9915 3496 50  0000 L CNN
-F 1 "100n" H 9915 3405 50  0000 L CNN
-F 2 "Capacitor_SMD:C_0603_1608Metric_Pad1.05x0.95mm_HandSolder" H 9838 3300 50  0001 C CNN
-F 3 "~" H 9800 3450 50  0001 C CNN
-	1    9800 3450
-	1    0    0    -1
-$EndComp
-Wire Wire Line
-	8800 3450 8800 3400
-Wire Wire Line
-	8800 3400 8875 3400
-Wire Wire Line
-	8800 3450 8800 3500
-Wire Wire Line
-	8800 3500 8875 3500
-Connection ~ 8800 3450
-$Comp
-L power:VCC #PWR0262
-U 1 1 5F813A57
-P 9175 3200
-F 0 "#PWR0262" H 9175 3050 50  0001 C CNN
-F 1 "VCC" H 9192 3373 50  0000 C CNN
-F 2 "" H 9175 3200 50  0001 C CNN
-F 3 "" H 9175 3200 50  0001 C CNN
-	1    9175 3200
+L power:VCC #PWR0105
+U 1 1 5FA70662
+P 5125 5800
+F 0 "#PWR0105" H 5125 5650 50  0001 C CNN
+F 1 "VCC" H 5142 5973 50  0000 C CNN
+F 2 "" H 5125 5800 50  0001 C CNN
+F 3 "" H 5125 5800 50  0001 C CNN
+	1    5125 5800
 	1    0    0    -1
 $EndComp
 $Comp
 L power:GND #PWR?
-U 1 1 5F813F7D
-P 9175 3675
-AR Path="/5F813F7D" Ref="#PWR?"  Part="1"
-AR Path="/5E4D7DB2/5F813F7D" Ref="#PWR0263"  Part="1"
-F 0 "#PWR0263" H 9175 3425 50  0001 C CNN
-F 1 "GND" H 9180 3502 50  0000 C CNN
-F 2 "" H 9175 3675 50  0001 C CNN
-F 3 "" H 9175 3675 50  0001 C CNN
-	1    9175 3675
+U 1 1 5FA70B36
+P 5125 7000
+AR Path="/5FA70B36" Ref="#PWR?"  Part="1"
+AR Path="/5E4D7DB2/5FA70B36" Ref="#PWR0111"  Part="1"
+F 0 "#PWR0111" H 5125 6750 50  0001 C CNN
+F 1 "GND" H 5130 6827 50  0000 C CNN
+F 2 "" H 5125 7000 50  0001 C CNN
+F 3 "" H 5125 7000 50  0001 C CNN
+	1    5125 7000
 	1    0    0    -1
 $EndComp
 Wire Wire Line
-	9175 3200 9175 3350
+	5125 5900 5125 5800
 Wire Wire Line
-	9175 3675 9175 3550
-$Comp
-L power:VCC #PWR0264
-U 1 1 5F815282
-P 9800 3200
-F 0 "#PWR0264" H 9800 3050 50  0001 C CNN
-F 1 "VCC" H 9817 3373 50  0000 C CNN
-F 2 "" H 9800 3200 50  0001 C CNN
-F 3 "" H 9800 3200 50  0001 C CNN
-	1    9800 3200
-	1    0    0    -1
-$EndComp
-$Comp
-L power:GND #PWR?
-U 1 1 5F8155B7
-P 9800 3675
-AR Path="/5F8155B7" Ref="#PWR?"  Part="1"
-AR Path="/5E4D7DB2/5F8155B7" Ref="#PWR0265"  Part="1"
-F 0 "#PWR0265" H 9800 3425 50  0001 C CNN
-F 1 "GND" H 9805 3502 50  0000 C CNN
-F 2 "" H 9800 3675 50  0001 C CNN
-F 3 "" H 9800 3675 50  0001 C CNN
-	1    9800 3675
-	1    0    0    -1
-$EndComp
-Wire Wire Line
-	9800 3200 9800 3300
-Wire Wire Line
-	9800 3675 9800 3600
+	5125 6900 5125 7000
 $EndSCHEMATC

Commit message: Track
Parts:
- R4, R6, R7: footprint Resistor_SMD:R_1206_3216Metric_Pad1.42x1.75mm_HandSolder -> Atari:R_Axial_DIN0207_L3.6mm_D2.2mm_P10.16mm_Horizontal
Changed lines of the file:
@@
 F 0 "R4" H 4620 3246 50  0000 L CNN
 F 1 "3k" H 4620 3155 50  0000 L CNN
-F 2 "Resistor_SMD:R_1206_3216Metric_Pad1.42x1.75mm_HandSolder" V 4480 3200 50  0001 C CNN
+F 2 "Atari:R_Axial_DIN0207_L3.6mm_D2.2mm_P10.16mm_Horizontal" V 4480 3200 50  0001 C CNN
 F 3 "~" H 4550 3200 50  0001 C CNN
 	1    4550 3200
@@
 F 0 "R6" H 4920 3246 50  0000 L CNN
 F 1 "3k" H 4920 3155 50  0000 L CNN
-F 2 "Resistor_SMD:R_1206_3216Metric_Pad1.42x1.75mm_HandSolder" V 4780 3200 50  0001 C CNN
+F 2 "Atari:R_Axial_DIN0207_L3.6mm_D2.2mm_P10.16mm_Horizontal" V 4780 3200 50  0001 C CNN
 F 3 "~" H 4850 3200 50  0001 C CNN
 	1    4850 3200
@@
 F 0 "R7" H 5220 3246 50  0000 L CNN
 F 1 "3k" H 5220 3155 50  0000 L CNN
-F 2 "Resistor_SMD:R_1206_3216Metric_Pad1.42x1.75mm_HandSolder" V 5080 3200 50  0001 C CNN
+F 2 "Atari:R_Axial_DIN0207_L3.6mm_D2.2mm_P10.16mm_Horizontal" V 5080 3200 50  0001 C CNN
 F 3 "~" H 5150 3200 50  0001 C CNN
 	1    5150 3200
