File: External Memory.sch (KiCad schematic (older format))
At the start: 13 parts, among them J7 SIMM_ON_OFF, U120 SIMM_exp_GAL, U121 DRAM_1MB_4bit, U122 DRAM_1MB_4bit, U123 74LS175, U124 74LS157

Commit message: memory track
Parts:
- U120: symbol Atari:SIMM_exp_GAL -> Atari-130XE-rescue:SIMM_exp_GAL-Atari
- U121, U122: symbol Atari:DRAM_1MB_4bit -> Atari-130XE-rescue:DRAM_1MB_4bit-Atari
Connections:
- net labels removed: RA8, RA9
- wire segments 59 -> 65
Changed lines of the file:
@@
 	2000 6875 2250 6875
 $Comp
-L Atari:SIMM_exp_GAL U120
+L Atari-130XE-rescue:SIMM_exp_GAL-Atari U120
 U 1 1 5F8607CE
 P 2225 3850
@@
 Connection ~ 825  1050
 $Comp
-L Atari:DRAM_1MB_4bit U121
+L Atari-130XE-rescue:DRAM_1MB_4bit-Atari U121
 U 1 1 5F87AE34
 P 8700 1875
+AR Path="/5F87AE34" Ref="U121"  Part="1"
+AR Path="/5E53A007/5F87AE34" Ref="U121"  Part="1"
 F 0 "U121" H 8700 2840 50  0000 C CNN
 F 1 "DRAM_1MB_4bit" H 8700 2749 50  0000 C CNN
@@
 $EndComp
 $Comp
-L Atari:DRAM_1MB_4bit U122
+L Atari-130XE-rescue:DRAM_1MB_4bit-Atari U122
 U 1 1 5F87D2A4
 P 8725 4275
+AR Path="/5F87D2A4" Ref="U122"  Part="1"
+AR Path="/5E53A007/5F87D2A4" Ref="U122"  Part="1"
 F 0 "U122" H 8725 5240 50  0000 C CNN
 F 1 "DRAM_1MB_4bit" H 8725 5149 50  0000 C CNN
@@
 Text GLabel 8250 2375 0    50   Input ~ 0
 RA7
-Text GLabel 8250 2475 0    50   Input ~ 0
-RA8
-Text GLabel 8250 2575 0    50   Input ~ 0
-RA9
 Text GLabel 8250 1375 0    50   Input ~ 0
 WRT
@@
 	7100 4550 7100 4875
 Wire Wire Line
-	7100 4875 8275 4875
+	7100 4875 7350 4875
 Wire Wire Line
 	6025 4850 6975 4850
@@
 	6975 4850 6975 4975
 Wire Wire Line
-	6975 4975 8275 4975
+	6975 4975 7475 4975
+Wire Wire Line
+	8250 2475 7350 2475
+Wire Wire Line
+	7350 2475 7350 4875
+Connection ~ 7350 4875
+Wire Wire Line
+	7350 4875 8275 4875
+Wire Wire Line
+	8250 2575 7475 2575
+Wire Wire Line
+	7475 2575 7475 4975
+Connection ~ 7475 4975
+Wire Wire Line
+	7475 4975 8275 4975
 $EndSCHEMATC

Commit message: Track
Parts:
- U120: footprint Package_DIP:DIP-24_W7.62mm_Socket -> Package_DIP:DIP-24_W7.62mm_Socket_LongPads
Changed lines of the file:
@@
 F 0 "U120" H 2225 5215 50  0000 C CNN
 F 1 "SIMM_exp_GAL" H 2225 5124 50  0000 C CNN
-F 2 "Package_DIP:DIP-24_W7.62mm_Socket" H 2225 3850 50  0001 C CNN
+F 2 "Package_DIP:DIP-24_W7.62mm_Socket_LongPads" H 2225 3850 50  0001 C CNN
 F 3 "" H 2225 3850 50  0001 C CNN
 	1    2225 3850

Commit message: Finished GND
Parts:
- added C98: 100uF, Capacitor_THT:CP_Radial_D6.3mm_P2.50mm, symbol Device:CP
Connections:
- net GND: now also C98.2
- net VCC: now also C98.1
Changed lines of the file:
@@
 Wire Wire Line
 	7475 4975 8275 4975
+$Comp
+L Device:CP C98
+U 1 1 5FC57288
+P 3150 7025
+F 0 "C98" H 3268 7071 50  0000 L CNN
+F 1 "100uF" H 3268 6980 50  0000 L CNN
+F 2 "Capacitor_THT:CP_Radial_D6.3mm_P2.50mm" H 3188 6875 50  0001 C CNN
+F 3 "~" H 3150 7025 50  0001 C CNN
+	1    3150 7025
+	1    0    0    -1
+$EndComp
+Wire Wire Line
+	3150 6875 2700 6875
+Connection ~ 2700 6875
+Wire Wire Line
+	3150 7175 2700 7175
+Connection ~ 2700 7175
 $EndSCHEMATC
