File: GTIA.sch (KiCad schematic (older format))
At the start: 87 parts, among them J2 DIN-5_180degree, J50 GTIA Fix, Q1 2N3904, Q2 2N3904, Q3 2N3904, Q6 2N3904, Q8 PN2222A, Q9 PN2222A, U11 74LS74, U113 74AHC1G08, U12 4050, U3 GTIA, U57 74HC14, U58 74LS175, Y2 4.43MHz

Commit message: Global rebuild up to 1mB
Parts:
- removed C250: 22pF, Capacitor_SMD:C_1206_3216Metric_Pad1.42x1.75mm_HandSolder, symbol Device:C
- removed C254, C255: 100nF, Capacitor_SMD:C_1206_3216Metric_Pad1.42x1.75mm_HandSolder, symbol Device:C
- removed D50: BAS316, Atari:D_SOD-323_HandSoldering, symbol Device:D
- removed J50: GTIA Fix, Connector_PinHeader_2.54mm:PinHeader_2x08_P2.54mm_Vertical, symbol Connector_Generic:Conn_02x08_Odd_Even
- removed R206: 1k, Resistor_SMD:R_1206_3216Metric_Pad1.42x1.75mm_HandSolder, symbol Device:R
- removed U57: 74HC14, Package_SO:SOIC-14_3.9x8.7mm_P1.27mm, symbol 74xx:74HC14
- removed U58: 74LS175, Package_SO:SOIC-16_3.9x9.9mm_P1.27mm, symbol 74xx:74LS175
Connections:
- net labels removed: AN0_FIX, AN1_FIX, AN2_FIX, GTIA_AN0, GTIA_AN1, GTIA_AN2, GTIA_NORM, GTIA_OSC, OSC_FIX
- wire segments 269 -> 239

Commit message: Track
Parts:
- removed U3: GTIA, Package_DIP:DIP-40_W15.24mm_LongPads, symbol Atari-130XE-rescue:GTIA-Atari
- added U3: GTIA, Package_DIP:DIP-40_W15.24mm_LongPads, symbol Atari:GTIA
Connections:
- net +5VA: now also U3.27 (VCC)
- net A0: now also U3.2 (A0)
- net A1: now also U3.1 (A1)
- net A2: now also U3.40 (A2)
- net A3: now also U3.39 (A3)
- net A4: now also U3.38 (A4)
- net AN0: now also U3.18 (AN0)
- net AN1: now also U3.19 (AN1)
- net AN2: now also U3.20 (AN2)
- net BELL: now also U3.15 (S3)
- net BO2: now also U3.30 (O2)
- net D0: now also U3.7 (D0)
- net D1: now also U3.6 (D1)
- net D2: now also U3.5 (D2)
- net D3: now also U3.4 (D3)
- net D4: now also U3.37 (D4)
- net D5: now also U3.36 (D5)
- net D6: now also U3.35 (D6)
- net D7: now also U3.34 (D7)
- net FO0: now also U3.29 (FO0)
- net GND: now also U3.3 (VSS)
- net GTIA: now also U3.32 (~CS)
- net HALT: now also U3.26 (HALT)
- net RD5: now also U3.11 (T3)
- net R\W: now also U3.33 (R/~W)
- net at R134.2: now also U3.12 (S0)
- net at R135.2: now also U3.13 (S1)
- net at R136.2: now also U3.14 (S2)
- net at Q6.3 (C), R70.1, R72.1: now also U3.16 (PAL)
- net at C48.2, RV1.2: now also U3.17 (CADJ)
- net at L6.1, R33.2, R41.2: now also U3.21 (COLOR)
- net at R44.2, U12.11: now also U3.22 (LUM1)
- net at R43.2, U12.5: now also U3.23 (LUM2)
- net at R42.2, U12.3: now also U3.24 (LUM3)
- net at U12.14: now also U3.25 (CSYNC)
- net at C206.1, FB3.1, U11.3 (C): now also U3.28 (OSC)
- net at R45.2, U12.7: now also U3.31 (LUM0)
- net at R132.1, U113.1: now also U3.8 (T0)
- net at R133.1, U113.2: now also U3.9 (T1)
Changed lines of the file:
@@
 Comment4 ""
 $EndDescr
-$Comp
-L Atari-130XE-rescue:GTIA-Atari U3
-U 1 1 5E53E87B
-P 4100 4450
-AR Path="/5E53E87B" Ref="U3"  Part="1"
-AR Path="/5E53E150/5E53E87B" Ref="U3"  Part="1"
-F 0 "U3" H 4100 6115 50  0000 C CNN
-F 1 "GTIA" H 4100 6024 50  0000 C CNN
-F 2 "Package_DIP:DIP-40_W15.24mm_LongPads" H 4100 4450 50  0001 C CNN
-F 3 "" H 4100 4450 50  0001 C CNN
-	1    4100 4450
-	1    0    0    -1
-$EndComp
 Text GLabel 3500 4550 0    50   Input ~ 0
 D0
@@
 Wire Wire Line
 	3650 10450 3650 10600
+$Comp
+L Atari:GTIA U3
+U 1 1 5F9F44AA
+P 4100 4450
+F 0 "U3" H 4100 6115 50  0000 C CNN
+F 1 "GTIA" H 4100 6024 50  0000 C CNN
+F 2 "Package_DIP:DIP-40_W15.24mm_LongPads" H 4100 4450 50  0001 C CNN
+F 3 "" H 4100 4450 50  0001 C CNN
+	1    4100 4450
+	1    0    0    -1
+$EndComp
 $EndSCHEMATC

Commit message: track
Parts:
- removed C107: 100nF, Capacitor_SMD:C_0603_1608Metric_Pad1.05x0.95mm_HandSolder, symbol Device:C
- removed U113: 74AHC1G08, Package_TO_SOT_SMD:SOT-23-5_HandSoldering, symbol 74xGxx:74AHC1G08
- added U10: 74LS08, Package_DIP:DIP-14_W7.62mm_Socket_LongPads, symbol 74xx:74LS08
Connections:
- net LP: now also U10.11
- net at R132.1, U3.8 (T0): now also U10.12
- net at R133.1, U3.9 (T1): now also U10.13
Changed lines of the file:
@@
 Wire Wire Line
 	7450 6375 7875 6375
-Text GLabel 6225 6875 2    50   Input ~ 0
+Text GLabel 6175 6825 2    50   Input ~ 0
 LP
-Wire Wire Line
-	6125 6875 6225 6875
 NoConn ~ 4700 4600
 $Comp
@@
 Wire Wire Line
 	14050 2050 13725 2050
-$Comp
-L 74xGxx:74AHC1G08 U113
-U 1 1 5F8309A6
-P 5875 6875
-F 0 "U113" H 5675 7050 50  0000 C CNN
-F 1 "74AHC1G08" H 5500 6725 50  0000 C CNN
-F 2 "Package_TO_SOT_SMD:SOT-23-5_HandSoldering" H 5875 6875 50  0001 C CNN
-F 3 "http://www.ti.com/lit/sg/scyt129e/scyt129e.pdf" H 5875 6875 50  0001 C CNN
-	1    5875 6875
-	1    0    0    -1
-$EndComp
-Wire Wire Line
-	5500 6225 5500 6825
-Wire Wire Line
-	5500 6825 5575 6825
-Connection ~ 5500 6225
 Wire Wire Line
 	5375 6375 5375 6925
@@
 	5375 6925 5575 6925
 Connection ~ 5375 6375
-$Comp
-L power:GND #PWR0105
-U 1 1 5F854381
-P 5875 7050
-F 0 "#PWR0105" H 5875 6800 50  0001 C CNN
-F 1 "GND" H 5880 6877 50  0000 C CNN
-F 2 "" H 5875 7050 50  0001 C CNN
-F 3 "" H 5875 7050 50  0001 C CNN
-	1    5875 7050
-	1    0    0    -1
-$EndComp
-$Comp
-L power:VCC #PWR0111
-U 1 1 5F8546B5
-P 5875 6675
-F 0 "#PWR0111" H 5875 6525 50  0001 C CNN
-F 1 "VCC" H 5892 6848 50  0000 C CNN
-F 2 "" H 5875 6675 50  0001 C CNN
-F 3 "" H 5875 6675 50  0001 C CNN
-	1    5875 6675
-	1    0    0    -1
-$EndComp
-Wire Wire Line
-	5875 7050 5875 6975
-Wire Wire Line
-	5875 6675 5875 6775
-$Comp
-L Device:C C107
-U 1 1 5F87A04E
-P 2425 10025
-F 0 "C107" H 2540 10071 50  0000 L CNN
-F 1 "100nF" H 2540 9980 50  0000 L CNN
-F 2 "Capacitor_SMD:C_0603_1608Metric_Pad1.05x0.95mm_HandSolder" H 2463 9875 50  0001 C CNN
-F 3 "~" H 2425 10025 50  0001 C CNN
-	1    2425 10025
-	1    0    0    -1
-$EndComp
-Wire Wire Line
-	2125 9875 2425 9875
-Wire Wire Line
-	2100 10175 2425 10175
 $Comp
 L Transistor_BJT:PN2222A Q8
@@
 	1    0    0    -1
 $EndComp
+$Comp
+L 74xx:74LS08 U10
+U 4 1 5FA87C92
+P 5875 6825
+F 0 "U10" H 5875 7150 50  0000 C CNN
+F 1 "74LS08" H 5875 7059 50  0000 C CNN
+F 2 "Package_DIP:DIP-14_W7.62mm_Socket_LongPads" H 5875 6825 50  0001 C CNN
+F 3 "http://www.ti.com/lit/gpn/sn74LS08" H 5875 6825 50  0001 C CNN
+	4    5875 6825
+	1    0    0    -1
+$EndComp
+Wire Wire Line
+	5500 6225 5500 6725
+Wire Wire Line
+	5500 6725 5575 6725
+Connection ~ 5500 6225
 $EndSCHEMATC

Commit message: Track
Connections:
- net +5VA: no longer U3.27 (VCC)
- net VCC: now also U3.27 (VCC)
Changed lines of the file:
@@
-	1    0    0    -1
-$EndComp
-$Comp
-L power:+5VA #PWR0235
-U 1 1 5E9AB3B8
-P 4925 5575
-F 0 "#PWR0235" H 4925 5425 50  0001 C CNN
-F 1 "+5VA" H 4940 5748 50  0000 C CNN
-F 2 "" H 4925 5575 50  0001 C CNN
-F 3 "" H 4925 5575 50  0001 C CNN
-	1    4925 5575
 	1    0    0    -1
 $EndComp
@@
 	5500 6725 5575 6725
 Connection ~ 5500 6225
+$Comp
+L power:VCC #PWR?
+U 1 1 5FABDB21
+P 4925 5575
+F 0 "#PWR?" H 4925 5425 50  0001 C CNN
+F 1 "VCC" H 4942 5748 50  0000 C CNN
+F 2 "" H 4925 5575 50  0001 C CNN
+F 3 "" H 4925 5575 50  0001 C CNN
+	1    4925 5575
+	1    0    0    -1
+$EndComp
 $EndSCHEMATC

Commit message: Track
Parts:
- Q1, Q2, Q3, Q6, Q8, Q9: footprint Package_TO_SOT_THT:TO-92 -> Package_TO_SOT_THT:TO-92_Inline
Changed lines of the file:
@@
 F 0 "Q6" H 7340 7971 50  0000 L CNN
 F 1 "2N3904" H 7340 7880 50  0000 L CNN
-F 2 "Package_TO_SOT_THT:TO-92" H 7350 7850 50  0001 L CIN
+F 2 "Package_TO_SOT_THT:TO-92_Inline" H 7350 7850 50  0001 L CIN
 F 3 "https://www.fairchildsemi.com/datasheets/2N/2N3904.pdf" H 7150 7925 50  0001 L CNN
 	1    7150 7925
@@
 F 0 "Q1" H 9615 7296 50  0000 L CNN
 F 1 "2N3904" H 9615 7205 50  0000 L CNN
-F 2 "Package_TO_SOT_THT:TO-92" H 9625 7175 50  0001 L CIN
+F 2 "Package_TO_SOT_THT:TO-92_Inline" H 9625 7175 50  0001 L CIN
 F 3 "https://www.fairchildsemi.com/datasheets/2N/2N3904.pdf" H 9425 7250 50  0001 L CNN
 	1    9425 7250
@@
 F 0 "Q3" H 11190 2446 50  0000 L CNN
 F 1 "2N3904" H 11190 2355 50  0000 L CNN
-F 2 "Package_TO_SOT_THT:TO-92" H 11200 2325 50  0001 L CIN
+F 2 "Package_TO_SOT_THT:TO-92_Inline" H 11200 2325 50  0001 L CIN
 F 3 "https://www.fairchildsemi.com/datasheets/2N/2N3904.pdf" H 11000 2400 50  0001 L CNN
 	1    11000 2400
@@
 F 0 "Q2" H 11290 5321 50  0000 L CNN
 F 1 "2N3904" H 11290 5230 50  0000 L CNN
-F 2 "Package_TO_SOT_THT:TO-92" H 11300 5200 50  0001 L CIN
+F 2 "Package_TO_SOT_THT:TO-92_Inline" H 11300 5200 50  0001 L CIN
 F 3 "https://www.fairchildsemi.com/datasheets/2N/2N3904.pdf" H 11100 5275 50  0001 L CNN
 	1    11100 5275
@@
 F 0 "Q8" H 10040 4296 50  0000 L CNN
 F 1 "PN2222A" H 10040 4205 50  0000 L CNN
-F 2 "Package_TO_SOT_THT:TO-92" H 10050 4175 50  0001 L CIN
+F 2 "Package_TO_SOT_THT:TO-92_Inline" H 10050 4175 50  0001 L CIN
 F 3 "http://www.fairchildsemi.com/ds/PN/PN2222A.pdf" H 9850 4250 50  0001 L CNN
 	1    9850 4250
@@
 F 0 "Q9" H 12390 3546 50  0000 L CNN
 F 1 "PN2222A" H 12390 3455 50  0000 L CNN
-F 2 "Package_TO_SOT_THT:TO-92" H 12400 3425 50  0001 L CIN
+F 2 "Package_TO_SOT_THT:TO-92_Inline" H 12400 3425 50  0001 L CIN
 F 3 "http://www.fairchildsemi.com/ds/PN/PN2222A.pdf" H 12200 3500 50  0001 L CNN
 	1    12200 3500

Commit message: Finished GND
Parts:
- added J12, J13: Conn_01x03, Connector_PinHeader_2.54mm:PinHeader_1x03_P2.54mm_Vertical, symbol Connector_Generic:Conn_01x03
- added J18, J19, J20, J21, J22, J23, J24, J25, J26, J27, J28, J29: Pin, Atari:Pin, symbol Atari:Pin
- C39: footprint Capacitor_SMD:C_1206_3216Metric_Pad1.42x1.75mm_HandSolder -> Capacitor_THT:C_Disc_D5.0mm_W2.5mm_P5.00mm
- R95, R96, R97, R98: footprint Resistor_SMD:R_1206_3216Metric_Pad1.42x1.75mm_HandSolder -> Atari:R_Axial_DIN0207_L3.6mm_D2.2mm_P10.16mm_Horizontal
Connections:
- net AUDIO: now also J13.1 (Pin_1)
- net CHROMA: now also J13.2 (Pin_2)
- net COMPOSITE: now also J12.2 (Pin_2)
- net GND: now also J12.3 (Pin_3), J13.3 (Pin_3), J18.1, J19.1, J20.1, J22.1, J26.1, J27.1, J28.1
- net MONO: now also J12.1 (Pin_1)
- net at C59.1, Y2.1: now also J21.1
- net at C111.1, L1.2, R71.1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: now also J23.1
- net at C44.1, Q1.2 (B), R35.2: now also J24.1
- net at C45.1, D2.1 (K), D3.2 (A): now also J25.1
- net at C39.1, Q8.1 (E), R95.1: now also J29.1
