File: PIA.sch (KiCad schematic (older format))
At the start: 33 parts, among them J4 Joystick_Port, J5 Joystick_Port, Q4 2N3906, U1 PIA

Commit message: Finished GND
Parts:
- Q4: footprint Package_TO_SOT_THT:TO-92 -> Package_TO_SOT_THT:TO-92_Inline
Changed lines of the file:
@@
 F 0 "Q4" H 8590 2496 50  0000 L CNN
 F 1 "2N3906" H 8590 2405 50  0000 L CNN
-F 2 "Package_TO_SOT_THT:TO-92" H 8600 2375 50  0001 L CIN
+F 2 "Package_TO_SOT_THT:TO-92_Inline" H 8600 2375 50  0001 L CIN
 F 3 "https://www.fairchildsemi.com/datasheets/2N/2N3906.pdf" H 8400 2450 50  0001 L CNN
 	1    8400 2450
