File: Freddie.sch (KiCad schematic (older format))
At the start: 25 parts, among them J3 Cartridge, U110 74AHC1G08, U111 74AHC1G08, U13 74LS138, U14 MMU, U9 Freddie, Y1 14,18757MHz

Commit message: track
Parts:
- removed C112, C113: 100n, Capacitor_SMD:C_0603_1608Metric_Pad1.05x0.95mm_HandSolder, symbol Device:C
- removed U110, U111: 74AHC1G08, Package_TO_SOT_SMD:SOT-23-5_HandSoldering, symbol 74xGxx:74AHC1G08
- added U10: 74LS08, Package_DIP:DIP-14_W7.62mm_Socket_LongPads, symbol 74xx:74LS08
- U13: footprint Package_DIP:DIP-16_W7.62mm_Socket -> Package_DIP:DIP-16_W7.62mm_Socket_LongPads
Connections:
- net BO2: now also U10.3
- net GTIA: now also U10.8
- net O2: now also U10.1
- net at R3.1: now also U10.2
- net at U13.15 (O0): now also U10.10, U10.9
Changed lines of the file:
@@
 F 0 "U13" H 8150 2500 50  0000 C CNN
 F 1 "74LS138" H 8550 2500 50  0000 C CNN
-F 2 "Package_DIP:DIP-16_W7.62mm_Socket" H 8350 2000 50  0001 C CNN
+F 2 "Package_DIP:DIP-16_W7.62mm_Socket_LongPads" H 8350 2000 50  0001 C CNN
 F 3 "http://www.ti.com/lit/gpn/sn74LS138" H 8350 2000 50  0001 C CNN
 	1    8350 2000
@@
 Wire Wire Line
 	8850 1700 9500 1700
-Text GLabel 10100 1700 2    50   Input ~ 0
+Text GLabel 10150 1700 2    50   Input ~ 0
 GTIA
 $Comp
@@
 Wire Wire Line
 	2350 7300 2350 7150
-$Comp
-L 74xGxx:74AHC1G08 U110
-U 1 1 5F834CAD
-P 1950 3525
-F 0 "U110" H 2125 3800 50  0000 C CNN
-F 1 "74AHC1G08" H 1700 3800 50  0000 C CNN
-F 2 "Package_TO_SOT_SMD:SOT-23-5_HandSoldering" H 1950 3525 50  0001 C CNN
-F 3 "http://www.ti.com/lit/sg/scyt129e/scyt129e.pdf" H 1950 3525 50  0001 C CNN
-	1    1950 3525
-	1    0    0    -1
-$EndComp
-$Comp
-L power:GND #PWR0120
-U 1 1 5F8357BE
-P 1950 3750
-F 0 "#PWR0120" H 1950 3500 50  0001 C CNN
-F 1 "GND" H 1955 3577 50  0000 C CNN
-F 2 "" H 1950 3750 50  0001 C CNN
-F 3 "" H 1950 3750 50  0001 C CNN
-	1    1950 3750
-	1    0    0    -1
-$EndComp
-Wire Wire Line
-	1950 3625 1950 3750
-$Comp
-L power:VCC #PWR0121
-U 1 1 5F8376CB
-P 1950 3175
-F 0 "#PWR0121" H 1950 3025 50  0001 C CNN
-F 1 "VCC" H 1967 3348 50  0000 C CNN
-F 2 "" H 1950 3175 50  0001 C CNN
-F 3 "" H 1950 3175 50  0001 C CNN
-	1    1950 3175
-	1    0    0    -1
-$EndComp
-Wire Wire Line
-	1950 3175 1950 3425
-Text GLabel 2200 3525 2    50   Input ~ 0
+Text GLabel 2325 3525 2    50   Input ~ 0
 BO2
 Wire Wire Line
@@
 Wire Wire Line
 	1450 3475 1650 3475
-$Comp
-L Device:C C112
-U 1 1 5F84C887
-P 2700 3525
-F 0 "C112" H 2815 3571 50  0000 L CNN
-F 1 "100n" H 2815 3480 50  0000 L CNN
-F 2 "Capacitor_SMD:C_0603_1608Metric_Pad1.05x0.95mm_HandSolder" H 2738 3375 50  0001 C CNN
-F 3 "~" H 2700 3525 50  0001 C CNN
-	1    2700 3525
-	1    0    0    -1
-$EndComp
-$Comp
-L power:VCC #PWR0122
-U 1 1 5F84D140
-P 2700 3175
-F 0 "#PWR0122" H 2700 3025 50  0001 C CNN
-F 1 "VCC" H 2717 3348 50  0000 C CNN
-F 2 "" H 2700 3175 50  0001 C CNN
-F 3 "" H 2700 3175 50  0001 C CNN
-	1    2700 3175
-	1    0    0    -1
-$EndComp
-$Comp
-L power:GND #PWR0123
-U 1 1 5F84D4A4
-P 2700 3775
-F 0 "#PWR0123" H 2700 3525 50  0001 C CNN
-F 1 "GND" H 2705 3602 50  0000 C CNN
-F 2 "" H 2700 3775 50  0001 C CNN
-F 3 "" H 2700 3775 50  0001 C CNN
-	1    2700 3775
-	1    0    0    -1
-$EndComp
-Wire Wire Line
-	2700 3375 2700 3175
-Wire Wire Line
-	2700 3775 2700 3675
-$Comp
-L 74xGxx:74AHC1G08 U111
-U 1 1 5F8518F1
-P 9850 1700
-F 0 "U111" H 10025 1975 50  0000 C CNN
-F 1 "74AHC1G08" H 9600 1975 50  0000 C CNN
-F 2 "Package_TO_SOT_SMD:SOT-23-5_HandSoldering" H 9850 1700 50  0001 C CNN
-F 3 "http://www.ti.com/lit/sg/scyt129e/scyt129e.pdf" H 9850 1700 50  0001 C CNN
-	1    9850 1700
-	1    0    0    -1
-$EndComp
-Wire Wire Line
-	9550 1650 9500 1650
-Wire Wire Line
-	9500 1650 9500 1700
-Wire Wire Line
-	9550 1750 9500 1750
-Wire Wire Line
-	9500 1750 9500 1700
-Connection ~ 9500 1700
-$Comp
-L power:VCC #PWR0124
-U 1 1 5F856467
-P 9850 1375
-F 0 "#PWR0124" H 9850 1225 50  0001 C CNN
-F 1 "VCC" H 9867 1548 50  0000 C CNN
-F 2 "" H 9850 1375 50  0001 C CNN
-F 3 "" H 9850 1375 50  0001 C CNN
-	1    9850 1375
-	1    0    0    -1
-$EndComp
-$Comp
-L power:GND #PWR0128
-U 1 1 5F85672D
-P 9850 2000
-F 0 "#PWR0128" H 9850 1750 50  0001 C CNN
-F 1 "GND" H 9855 1827 50  0000 C CNN
-F 2 "" H 9850 2000 50  0001 C CNN
-F 3 "" H 9850 2000 50  0001 C CNN
-	1    9850 2000
-	1    0    0    -1
-$EndComp
-Wire Wire Line
-	9850 1375 9850 1600
-Wire Wire Line
-	9850 2000 9850 1800
-$Comp
-L Device:C C113
-U 1 1 5F859D5A
-P 10725 1700
-F 0 "C113" H 10840 1746 50  0000 L CNN
-F 1 "100n" H 10840 1655 50  0000 L CNN
-F 2 "Capacitor_SMD:C_0603_1608Metric_Pad1.05x0.95mm_HandSolder" H 10763 1550 50  0001 C CNN
-F 3 "~" H 10725 1700 50  0001 C CNN
-	1    10725 1700
-	1    0    0    -1
-$EndComp
-$Comp
-L power:VCC #PWR0129
-U 1 1 5F85A45D
-P 10725 1375
-F 0 "#PWR0129" H 10725 1225 50  0001 C CNN
-F 1 "VCC" H 10742 1548 50  0000 C CNN
-F 2 "" H 10725 1375 50  0001 C CNN
-F 3 "" H 10725 1375 50  0001 C CNN
-	1    10725 1375
-	1    0    0    -1
-$EndComp
-Wire Wire Line
-	10725 1375 10725 1550
-$Comp
-L power:GND #PWR0130
-U 1 1 5F85C52A
-P 10725 2000
-F 0 "#PWR0130" H 10725 1750 50  0001 C CNN
-F 1 "GND" H 10730 1827 50  0000 C CNN
-F 2 "" H 10725 2000 50  0001 C CNN
-F 3 "" H 10725 2000 50  0001 C CNN
-	1    10725 2000
-	1    0    0    -1
-$EndComp
-Wire Wire Line
-	10725 1850 10725 2000
 Text GLabel 9000 4050 2    50   Input ~ 0
 BE
@@
 Wire Wire Line
 	5975 3700 5975 3800
+$Comp
+L 74xx:74LS08 U10
+U 1 1 5FA753F3
+P 2025 3525
+F 0 "U10" H 2025 3850 50  0000 C CNN
+F 1 "74LS08" H 2025 3759 50  0000 C CNN
+F 2 "Package_DIP:DIP-14_W7.62mm_Socket_LongPads" H 2025 3525 50  0001 C CNN
+F 3 "http://www.ti.com/lit/gpn/sn74LS08" H 2025 3525 50  0001 C CNN
+	1    2025 3525
+	1    0    0    -1
+$EndComp
+Wire Wire Line
+	1650 3475 1650 3425
+Wire Wire Line
+	1650 3425 1725 3425
+Wire Wire Line
+	1650 3575 1650 3625
+Wire Wire Line
+	1650 3625 1725 3625
+$Comp
+L 74xx:74LS08 U10
+U 3 1 5FA7E8F4
+P 9850 1700
+F 0 "U10" H 9850 2025 50  0000 C CNN
+F 1 "74LS08" H 9850 1934 50  0000 C CNN
+F 2 "Package_DIP:DIP-14_W7.62mm_Socket_LongPads" H 9850 1700 50  0001 C CNN
+F 3 "http://www.ti.com/lit/gpn/sn74LS08" H 9850 1700 50  0001 C CNN
+	3    9850 1700
+	1    0    0    -1
+$EndComp
+Wire Wire Line
+	9500 1700 9500 1600
+Wire Wire Line
+	9500 1600 9550 1600
+Wire Wire Line
+	9500 1700 9500 1800
+Wire Wire Line
+	9500 1800 9550 1800
+Connection ~ 9500 1700
 $EndSCHEMATC

Commit message: Finished GND
Parts:
- added J14: Conn_01x06, Connector_PinHeader_2.54mm:PinHeader_1x06_P2.54mm_Vertical, symbol Connector_Generic:Conn_01x06
- added J16: Conn_01x05, Connector_PinHeader_2.54mm:PinHeader_1x05_P2.54mm_Vertical, symbol Connector_Generic:Conn_01x05
- added J17: Conn_01x04, Connector_PinHeader_2.54mm:PinHeader_1x04_P2.54mm_Vertical, symbol Connector_Generic:Conn_01x04
- R16, R17: footprint Resistor_THT:R_Axial_DIN0207_L6.3mm_D2.5mm_P10.16mm_Horizontal -> Atari:R_Axial_DIN0207_L3.6mm_D2.2mm_P10.16mm_Horizontal
Connections:
- net BO2: now also J17.4 (Pin_4)
- net CAS: now also J14.4 (Pin_4)
- net CASINH: now also J16.3 (Pin_3)
- net EXTSEL: now also J16.2 (Pin_2)
- net GND: now also J14.3 (Pin_3), J16.5 (Pin_5), J17.1 (Pin_1)
- net O2: now also J16.4 (Pin_4), J17.3 (Pin_3)
- net OSC: now also J14.2 (Pin_2)
- net RAS: now also J14.6 (Pin_6)
- net R\W: now also J14.1 (Pin_1)
- net WRT: now also J14.5 (Pin_5)
- net at C22.1, R17.2, U9.2 (CLK)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: now also J16.1 (Pin_1)
- new net O0: J17.2 (Pin_2)
Changed lines of the file:
@@
 F 0 "R16" V 2143 1250 50  0000 C CNN
 F 1 "240" V 2234 1250 50  0000 C CNN
-F 2 "Resistor_THT:R_Axial_DIN0207_L6.3mm_D2.5mm_P10.16mm_Horizontal" V 2280 1250 50  0001 C CNN
+F 2 "Atari:R_Axial_DIN0207_L3.6mm_D2.2mm_P10.16mm_Horizontal" V 2280 1250 50  0001 C CNN
 F 3 "~" H 2350 1250 50  0001 C CNN
 	1    2350 1250
@@
 F 0 "R17" V 2143 2000 50  0000 C CNN
 F 1 "1M" V 2234 2000 50  0000 C CNN
-F 2 "Resistor_THT:R_Axial_DIN0207_L6.3mm_D2.5mm_P10.16mm_Horizontal" V 2280 2000 50  0001 C CNN
+F 2 "Atari:R_Axial_DIN0207_L3.6mm_D2.2mm_P10.16mm_Horizontal" V 2280 2000 50  0001 C CNN
 F 3 "~" H 2350 2000 50  0001 C CNN
 	1    2350 2000
@@
 	9500 1800 9550 1800
 Connection ~ 9500 1700
+$Comp
+L Connector_Generic:Conn_01x06 J14
+U 1 1 5FC9F389
+P 3125 4725
+F 0 "J14" H 3205 4717 50  0000 L CNN
+F 1 "Conn_01x06" H 3205 4626 50  0000 L CNN
+F 2 "Connector_PinHeader_2.54mm:PinHeader_1x06_P2.54mm_Vertical" H 3125 4725 50  0001 C CNN
+F 3 "~" H 3125 4725 50  0001 C CNN
+	1    3125 4725
+	1    0    0    -1
+$EndComp
+Text GLabel 2925 4525 0    50   Input ~ 0
+R\W
+Text GLabel 2925 4625 0    50   Input ~ 0
+OSC
+Text GLabel 2925 4825 0    50   Input ~ 0
+CAS
+Text GLabel 2925 4925 0    50   Input ~ 0
+WRT
+Text GLabel 2925 5025 0    50   Input ~ 0
+RAS
+$Comp
+L power:GND #PWR0128
+U 1 1 5FCA0518
+P 2550 5725
+F 0 "#PWR0128" H 2550 5475 50  0001 C CNN
+F 1 "GND" H 2555 5552 50  0000 C CNN
+F 2 "" H 2550 5725 50  0001 C CNN
+F 3 "" H 2550 5725 50  0001 C CNN
+	1    2550 5725
+	1    0    0    -1
+$EndComp
+Wire Wire Line
+	2925 4725 2550 4725
+$Comp
+L Connector_Generic:Conn_01x05 J16
+U 1 1 5FCAEA58
+P 3125 4125
+F 0 "J16" H 3205 4167 50  0000 L CNN
+F 1 "Conn_01x05" H 3205 4076 50  0000 L CNN
+F 2 "Connector_PinHeader_2.54mm:PinHeader_1x05_P2.54mm_Vertical" H 3125 4125 50  0001 C CNN
+F 3 "~" H 3125 4125 50  0001 C CNN
+	1    3125 4125
+	1    0    0    -1
+$EndComp
+Wire Wire Line
+	2650 2200 2650 3925
+Wire Wire Line
+	2650 3925 2925 3925
+Connection ~ 2650 2200
+Text GLabel 2925 4025 0    50   Input ~ 0
+EXTSEL
+Text GLabel 2925 4125 0    50   Input ~ 0
+CASINH
+Text GLabel 2925 4225 0    50   Input ~ 0
+O2
+Wire Wire Line
+	2925 4325 2550 4325
+Wire Wire Line
+	2550 4325 2550 4725
+Connection ~ 2550 4725
+$Comp
+L Connector_Generic:Conn_01x04 J17
+U 1 1 5FCBC25F
+P 3125 5400
+F 0 "J17" H 3205 5392 50  0000 L CNN
+F 1 "Conn_01x04" H 3205 5301 50  0000 L CNN
+F 2 "Connector_PinHeader_2.54mm:PinHeader_1x04_P2.54mm_Vertical" H 3125 5400 50  0001 C CNN
+F 3 "~" H 3125 5400 50  0001 C CNN
+	1    3125 5400
+	1    0    0    -1
+$EndComp
+Wire Wire Line
+	2550 4725 2550 5300
+Text GLabel 2925 5400 0    50   Input ~ 0
+O0
+Text GLabel 2925 5600 0    50   Input ~ 0
+BO2
+Text GLabel 2925 5500 0    50   Input ~ 0
+O2
+Wire Wire Line
+	2925 5300 2550 5300
+Connection ~ 2550 5300
+Wire Wire Line
+	2550 5300 2550 5725
 $EndSCHEMATC

Commit message: Gerber
Parts:
- R1: footprint Resistor_SMD:R_1206_3216Metric_Pad1.42x1.75mm_HandSolder -> Atari:R_Axial_DIN0207_L3.6mm_D2.2mm_P10.16mm_Horizontal
Changed lines of the file:
@@
 F 0 "R1" H 6130 1554 50  0000 R CNN
 F 1 "3k" H 6130 1645 50  0000 R CNN
-F 2 "Resistor_SMD:R_1206_3216Metric_Pad1.42x1.75mm_HandSolder" V 6130 1600 50  0001 C CNN
+F 2 "Atari:R_Axial_DIN0207_L3.6mm_D2.2mm_P10.16mm_Horizontal" V 6130 1600 50  0001 C CNN
 F 3 "~" H 6200 1600 50  0001 C CNN
 	1    6200 1600
