File: POKEY.sch (KiCad schematic (older format))
At the start: 51 parts, among them J15 SIO_Port, J6 Keyboard, U5 POKEY, U62 4051, U63 4051

Commit message: Gerber
Parts:
- C34: footprint Capacitor_SMD:CP_Elec_6.3x5.3 -> Capacitor_THT:CP_Radial_D5.0mm_P2.00mm
Changed lines of the file:
@@
 F 0 "C34" H 1918 6646 50  0000 L CNN
 F 1 "22uF" H 1918 6555 50  0000 L CNN
-F 2 "Capacitor_SMD:CP_Elec_6.3x5.3" H 1838 6450 50  0001 C CNN
+F 2 "Capacitor_THT:CP_Radial_D5.0mm_P2.00mm" H 1838 6450 50  0001 C CNN
 F 3 "~" H 1800 6600 50  0001 C CNN
 	1    1800 6600
